File: Fragaria-2.0/fragaria-extend/fragaria-extend.kicad_pcb (KiCad board)
At the start: 2 copper layers, 40 x 75 mm, 82 parts, among them CN1 AS0BC21-S40BB-7H, CN2 PJ-327A_5JJ, J1 Conn_01x04, J2 Conn_01x04, J3 Conn_01x06, J4 Conn_01x04, J5 Conn_01x04, SW1 MSK12C02, U1 XC6206P302MR_C347375, U2 AMS1117-3.3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

Commit message: Align numbering specifications
Parts:
- C1, C13, C14, C16, C19, C5: value 100nF -> 0.1uF
Changed lines of the file:
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@@
         (effects (font (size 1 1) (thickness 0.15)))
     )
-    (fp_text value "100nF" (at 0 1.43 90) (layer "F.Fab") hide
+    (fp_text value "0.1uF" (at 0 1.43 90) (layer "F.Fab") hide
         (effects (font (size 1 1) (thickness 0.15)))
     )
@@
         (effects (font (size 1 1) (thickness 0.15)))
     )
-    (fp_text value "100nF" (at 0 1.43) (layer "F.Fab") hide
+    (fp_text value "0.1uF" (at 0 1.43) (layer "F.Fab") hide
         (effects (font (size 1 1) (thickness 0.15)))
     )
@@
         (effects (font (size 1 1) (thickness 0.15)))
     )
-    (fp_text value "100nF" (at 0 1.43) (layer "F.Fab") hide
+    (fp_text value "0.1uF" (at 0 1.43) (layer "F.Fab") hide
         (effects (font (size 1 1) (thickness 0.15)))
     )
@@
         (effects (font (size 1 1) (thickness 0.15)))
     )
-    (fp_text value "100nF" (at 0 1.43 90) (layer "F.Fab") hide
+    (fp_text value "0.1uF" (at 0 1.43 90) (layer "F.Fab") hide
         (effects (font (size 1 1) (thickness 0.15)))
     )
@@
         (effects (font (size 1 1) (thickness 0.15)) (justify mirror))
     )
-    (fp_text value "100nF" (at 0 -1.43) (layer "B.Fab") hide
+    (fp_text value "0.1uF" (at 0 -1.43) (layer "B.Fab") hide
         (effects (font (size 1 1) (thickness 0.15)) (justify mirror))
     )
@@
         (effects (font (size 1 1) (thickness 0.15)) (justify mirror))
     )
-    (fp_text value "100nF" (at 0 -1.43) (layer "B.Fab") hide
+    (fp_text value "0.1uF" (at 0 -1.43) (layer "B.Fab") hide
         (effects (font (size 1 1) (thickness 0.15)) (justify mirror))
     )
