File: Fragaria-2.0/fragaria-extend/fragaria-extend.kicad_sch (KiCad schematic)
At the start: 81 parts, among them CN1 AS0BC21-S40BB-7H, CN2 PJ-327A_5JJ, J1 Conn_01x04, J2 Conn_01x04, J3 Conn_01x06, J4 Conn_01x04, J5 Conn_01x04, SW1 MSK12C02, U2 AMS1117-3.3, U3 SL2.1A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

Commit message: Align numbering specifications
Parts:
- C1, C13, C14, C16, C19, C5: value 100nF -> 0.1uF
Changed lines of the file:
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@@
       (effects (font (size 1.27 1.27)) (justify left))
     )
-    (property "Value" "100nF" (at 20.32 161.925 0)
+    (property "Value" "0.1uF" (at 20.32 161.925 0)
       (effects (font (size 1.27 1.27)) (justify left))
     )
@@
       (effects (font (size 1.27 1.27)))
     )
-    (property "Value" "100nF" (at 166.37 103.505 90)
+    (property "Value" "0.1uF" (at 166.37 103.505 90)
       (effects (font (size 1.27 1.27)))
     )
@@
       (effects (font (size 1.27 1.27)) (justify left))
     )
-    (property "Value" "100nF" (at 56.515 161.925 0)
+    (property "Value" "0.1uF" (at 56.515 161.925 0)
       (effects (font (size 1.27 1.27)) (justify left))
     )
@@
       (effects (font (size 1.27 1.27)) (justify left))
     )
-    (property "Value" "100nF" (at 224.79 36.83 0)
+    (property "Value" "0.1uF" (at 224.79 36.83 0)
       (effects (font (size 1.27 1.27)) (justify left))
     )
@@
       (effects (font (size 1.27 1.27)))
     )
-    (property "Value" "100nF" (at 166.37 126.365 90)
+    (property "Value" "0.1uF" (at 166.37 126.365 90)
       (effects (font (size 1.27 1.27)))
     )
@@
       (effects (font (size 1.27 1.27)))
     )
-    (property "Value" "100nF" (at 186.69 132.715 90)
+    (property "Value" "0.1uF" (at 186.69 132.715 90)
       (effects (font (size 1.27 1.27)))
     )
